File: TransceiverRF/Conector_EDU-CIAA.sch (KiCad schematic (older format))
At the start: 1 part

Commit message: agrego pcb
Connections:
- net Csn_1101: now also XA1.9 (ADC3); no longer XA1.76 (GPIO5)
- net Csn_2500: now also XA1.80 (GPIO8); no longer XA1.73 (GPIO4)
- net Earth: no longer XA1.57 (GND)
- net GDO1(opcional)_CC1101: now also XA1.11 (ADC2); no longer XA1.72 (GPIO1)
- net GDO1(opcional)_CC2500: now also XA1.78 (GPIO7); no longer XA1.69 (GPIO0)
- net GDO2(opcional)_CC1101: now also XA1.13 (ADC1); no longer XA1.74 (GPIO3)
- net SCLK_1101: now also XA1.25 (rs232TXD); no longer XA1.55 (ethRCLCK)
- net SI_CC1101: now also XA1.29 (canTD); no longer XA1.46 (ethTXEN)
- net SO_CC1101: now also XA1.15 (DAC); no longer XA1.44 (ethRXD1)
- no-connect marks 45 -> 46
Other:
- note removed: "Conectores EDU-CIAA-NXP"
Changed lines of the file:
@@
 encoding utf-8
 Sheet 4 4
-Title ""
-Date ""
-Rev ""
-Comp ""
+Title "Conectores"
+Date "2017-11-12"
+Rev "Gonzalo 1.1"
+Comp "Poncho CIAA"
 Comment1 ""
 Comment2 ""
@@
 	3800 3950 3200 3950
 Connection ~ 3200 4250
-Wire Wire Line
-	3800 3850 3750 3850
-Wire Wire Line
-	3750 3850 3750 3950
-Connection ~ 3750 3950
 Wire Wire Line
 	3800 4250 3750 4250
@@
 NoConn ~ 6950 4650
 NoConn ~ 6950 4550
-NoConn ~ 6950 4450
 NoConn ~ 6950 4350
-NoConn ~ 6950 4250
 NoConn ~ 6950 4150
 NoConn ~ 6950 3850
-NoConn ~ 6950 3750
-NoConn ~ 6950 3650
-NoConn ~ 6950 3550
-NoConn ~ 6950 3450
 NoConn ~ 6950 3350
 NoConn ~ 6950 3150
@@
 Text HLabel 5300 3850 2    60   Input ~ 0
 SO_CC2500
-Text HLabel 3050 4450 0    60   Input ~ 0
+Text HLabel 5150 4850 2    60   Input ~ 0
 GDO1(opcional)_CC2500
 Text HLabel 3050 4550 0    60   Input ~ 0
 GDO2(opcional)_CC2500
-Text HLabel 3050 4650 0    60   Input ~ 0
+Text HLabel 5150 4950 2    60   Input ~ 0
 Csn_2500
-Text HLabel 5300 3250 2    60   Input ~ 0
+Text HLabel 6750 4450 0    60   Input ~ 0
 SI_CC1101
-Text HLabel 2900 3750 0    60   Input ~ 0
+Text HLabel 6700 4250 0    60   Input ~ 0
 SCLK_1101
-Text HLabel 5300 3150 2    60   Input ~ 0
+Text HLabel 6800 3750 0    60   Input ~ 0
 SO_CC1101
-Text HLabel 5350 4550 2    60   Input ~ 0
+Text HLabel 6800 3550 0    60   Input ~ 0
 GDO1(opcional)_CC1101
-Text HLabel 5350 4650 2    60   Input ~ 0
+Text HLabel 6800 3650 0    60   Input ~ 0
 GDO2(opcional)_CC1101
-Text HLabel 5350 4750 2    60   Input ~ 0
+Text HLabel 6800 3450 0    60   Input ~ 0
 Csn_1101
 Wire Wire Line
@@
 	5000 3950 5300 3950
 Wire Wire Line
-	3050 4450 3800 4450
-Wire Wire Line
 	3050 4550 3800 4550
-Wire Wire Line
-	3050 4650 3800 4650
-Wire Wire Line
-	5000 3150 5300 3150
-Wire Wire Line
-	5000 3250 5300 3250
-Wire Wire Line
-	5000 4550 5350 4550
-Wire Wire Line
-	5000 4650 5350 4650
-Wire Wire Line
-	5000 4750 5350 4750
-Text Notes 7350 7500 0    60   ~ 0
-Conectores EDU-CIAA-NXP
-NoConn ~ 5000 4850
-NoConn ~ 5000 4950
+NoConn ~ 3800 4450
+NoConn ~ 3800 4650
 NoConn ~ 6950 3950
 NoConn ~ 6950 4050
 NoConn ~ 3800 4750
 NoConn ~ 6950 3250
-Wire Wire Line
-	2900 3750 3800 3750
 $Comp
 L Earth #PWR042
@@
 Wire Wire Line
 	1800 1850 1800 1550
-$Comp
-L PWR_FLAG #FLG045
-U 1 1 59F3F6D9
-P 2350 1550
-F 0 "#FLG045" H 2350 1625 50  0001 C CNN
-F 1 "PWR_FLAG" H 2350 1700 50  0000 C CNN
-F 2 "" H 2350 1550 50  0001 C CNN
-F 3 "" H 2350 1550 50  0001 C CNN
-	1    2350 1550
-	1    0    0    -1
-$EndComp
-$Comp
-L +3.3V #PWR046
-U 1 1 59F3F6F1
-P 2800 1550
-F 0 "#PWR046" H 2800 1400 50  0001 C CNN
-F 1 "+3.3V" H 2800 1690 50  0000 C CNN
-F 2 "" H 2800 1550 50  0001 C CNN
-F 3 "" H 2800 1550 50  0001 C CNN
-	1    2800 1550
-	1    0    0    -1
-$EndComp
-Wire Wire Line
-	2350 1550 2800 1550
+NoConn ~ 5000 3150
+NoConn ~ 5000 3250
+NoConn ~ 5000 4550
+NoConn ~ 5000 4650
+NoConn ~ 5000 4750
+Wire Wire Line
+	6800 3450 6950 3450
+Wire Wire Line
+	6800 3550 6950 3550
+Wire Wire Line
+	6800 3650 6950 3650
+Wire Wire Line
+	6750 4450 6950 4450
+Wire Wire Line
+	6700 4250 6950 4250
+NoConn ~ 3800 3750
+Wire Wire Line
+	6800 3750 6950 3750
+Wire Wire Line
+	5000 4950 5150 4950
+Wire Wire Line
+	5000 4850 5150 4850
+NoConn ~ 3800 3850
 $EndSCHEMATC
