File: TransceiverRF/TransceiverRF.sch (KiCad schematic (older format))
At the start: 0 parts

Commit message: agrego pcb
Other:
- note removed: "21 SEP 2017"
- note removed: "Trnsceiver RF"
Changed lines of the file:
@@
 encoding utf-8
 Sheet 1 4
-Title ""
-Date ""
-Rev ""
-Comp ""
+Title "TransceiverRF"
+Date "2017-11-12"
+Rev "Gonzalo 1.1"
+Comp "Poncho CIAA"
 Comment1 ""
 Comment2 ""
@@
 Comment4 ""
 $EndDescr
-Text Notes 7350 7500 0    60   ~ 0
-Trnsceiver RF
-Text Notes 8100 7650 0    60   ~ 0
-21 SEP 2017
 $Sheet
 S 2600 4150 1650 1000
@@
 F3 "SI_CC1101" I R 4250 4250 60
 F4 "SO_CC1101" I R 4250 4550 60
-F5 "GDO2(opcional)_CC1101" I R 4250 4700 60
-F6 "GDO1(opcional)_CC1101" I R 4250 4850 60
+F5 "GDO2(opcional)_CC1101" I R 4250 4850 60
+F6 "GDO1(opcional)_CC1101" I R 4250 4700 60
 F7 "CSn_CC1101" I R 4250 5000 60
 $EndSheet
