File: TransceiverRF/cc1101.sch (KiCad schematic (older format))
At the start: 24 parts, among them U1 CC1101, U2 CON_SMA, Y1 26 MHz

Commit message: agrego pcb
Other:
- note removed: "21 SEP 2017"
- note removed: "CC1101 Transceiver 433 MHz"
Changed lines of the file:
@@
 encoding utf-8
 Sheet 2 4
-Title ""
-Date ""
-Rev ""
-Comp ""
+Title "cc1101 Transceiver 433 MHz"
+Date "2017-11-12"
+Rev "Gonzalo 1.1"
+Comp "Poncho CIAA"
 Comment1 ""
 Comment2 ""
@@
 Comment4 ""
 $EndDescr
-Text Notes 7350 7500 0    60   ~ 0
-CC1101 Transceiver 433 MHz
-Text Notes 8100 7650 0    60   ~ 0
-21 SEP 2017
 $Comp
 L C C?
@@
 	5450 2400 5450 3100
 Wire Wire Line
-	6350 2850 6350 4900
+	6350 4900 6350 2850
 Wire Wire Line
 	6350 2850 5450 2850
 Connection ~ 5450 2850
 Connection ~ 6350 3600
-Wire Wire Line
-	6350 4900 5650 4900
 Connection ~ 6350 3800
 Connection ~ 6350 4400
@@
 Wire Wire Line
 	4050 2400 4050 2350
+Wire Wire Line
+	5650 4900 5650 5000
+Wire Wire Line
+	5650 5000 5950 5000
+Wire Wire Line
+	5950 5000 5950 4900
+Wire Wire Line
+	5950 4900 6350 4900
 $EndSCHEMATC
