File: TransceiverRF/cc2500.sch (KiCad schematic (older format))
At the start: 23 parts, among them U3 CC2500, U4 CON_SMA, Y2 26 MHz

Commit message: agrego pcb
Other:
- note removed: "CC2500 Transceiver 2.4 GHz"
Changed lines of the file:
@@
 encoding utf-8
 Sheet 3 4
-Title ""
-Date ""
-Rev ""
-Comp ""
+Title "cc2500 Transceiver 2.4 GHz"
+Date "2017-11-12"
+Rev "Gonzalo 1.1"
+Comp "Poncho CIAA"
 Comment1 ""
 Comment2 ""
@@
 Wire Wire Line
 	5300 2050 5300 2100
-Text Notes 7350 7500 0    60   ~ 0
-CC2500 Transceiver 2.4 GHz
 $Comp
 L +3.3V #PWR029
